File: schematic/schematic.kicad_sch (KiCad schematic)
At the start: 34 parts

Commit message: Schematic update
Parts:
- removed R? (x5): R_Small, symbol Device:R_Small
- added N? (x6): ITT5870S, symbol ITT5870S:ITT5870S
- added R? (x5): R_Small, symbol Device:R_Small
Connections:
- net at R?.1: now also N?. (dpR)
- new net: N?. (dpR), R?.1 (x5)
- no-connect marks 1 -> 13
Other:
- moved on the sheet: C?, D?, J?, Li-Po, R?, SW?, U?, Y?

Commit message: Updated schematic
Parts:
- removed N? (x5): ITT5870S, symbol ITT5870S:ITT5870S
- removed R? (x5): R_Small, symbol Device:R_Small
- removed SW? (x2): SW_Push, symbol Switch:SW_Push
- removed U? (x5): 74141, symbol 74xx_IEEE:74141
- added N? (x5): ITT5870S, symbol ITT5870S:ITT5870S
- added R? (x5): R_Small, symbol Device:R_Small
- added SW? (x2): SW_Push, symbol Switch:SW_Push
- added U?: HV_180V, symbol Regulator_Linear:L7805
- added U? (x5): 74141, symbol 74xx_IEEE:74141
Connections:
- net Led1 is gone; now on an unnamed net: U?.24 (PC2)
- net Led2 is gone; now on an unnamed net: U?.25 (PC3)
- net GND: now also SW?.2, SW?.2, SW?.2, U?.12 (GND), U?.12 (GND), U?.12 (GND), U?.12 (GND), U?.12 (GND), U?.2 (GND); no longer SW?.1
- net VCC: now also U?.5 (VCC), U?.5 (VCC), U?.5 (VCC), U?.5 (VCC), U?.5 (VCC)
- net at C?.1, J?.1, U?.1 (IN): now also U?.1 (IN)
- net K9: now reaches N?. (dpR)
- net K9: now also U?.2 (~{Q9}), N?. (dpR), N?. (dpR), N?. (dpR), N?. (dpR), N?. (dpR), U?.2 (~{Q9}), U?.2 (~{Q9}), U?.2 (~{Q9}), U?.2 (~{Q9}), U?.2 (~{Q9})
- net U1_1: now reaches U?.1 (QB)
- net U1_1: now also U?.6 (B)
- net U1_0: now reaches U?.15 (QA)
- net U1_0: now also U?.3 (A)
- net U1_2: now reaches U?.2 (QC)
- net U1_2: now also U?.7 (C)
- net U1_3: now reaches U?.3 (QD)
- net U1_3: now also U?.4 (D)
- net U1_4: now reaches U?.4 (QE)
- net U1_4: now also U?.3 (A)
- net U1_5: now reaches U?.5 (QF)
- net U1_5: now also U?.6 (B)
- net U1_6: now reaches U?.6 (QG)
- net U1_6: now also U?.7 (C)
- net U1_7: now reaches U?.7 (QH)
- net U1_7: now also U?.4 (D)
- net HV: now reaches R?.2
- net HV: now also R?.2, R?.2, R?.2, R?.2, R?.2, U?.3 (OUT)
- net U3_1: now reaches U?.1 (QB)
- net U3_1: now also U?.6 (B)
- net U3_0: now reaches U?.15 (QA)
- net U3_0: now also U?.3 (A)
- net U3_2: now reaches U?.2 (QC)
- net U3_2: now also U?.7 (C)
- net U3_3: now reaches U?.3 (QD)
- net U3_3: now also U?.4 (D)
- net U3_4: now reaches U?.4 (QE)
- net U3_4: now also U?.3 (A)
- net U3_5: now reaches U?.5 (QF)
- net U3_5: now also U?.6 (B)
- net U3_6: now reaches U?.6 (QG)
- net U3_6: now also U?.7 (C)
- net U3_7: now reaches U?.7 (QH)
- net U3_7: now also U?.4 (D)
- net U2_1: now reaches U?.1 (QB)
- net U2_1: now also U?.6 (B)
- net U2_0: now reaches U?.15 (QA)
- net U2_0: now also U?.3 (A)
- net U2_2: now reaches U?.2 (QC)
- net U2_2: now also U?.7 (C)
- net U2_3: now reaches U?.3 (QD)
- net U2_3: now also U?.4 (D)
- net U2_4: now reaches U?.4 (QE)
- net U2_4: now also U?.3 (A)
- net U2_5: now reaches U?.5 (QF)
- net U2_5: now also U?.6 (B)
- net U2_6: now reaches U?.6 (QG)
- net U2_6: now also U?.7 (C)
- net U2_7: now reaches U?.7 (QH)
- net U2_7: now also U?.4 (D)
- net K8: now reaches U?.1 (~{Q8})
- net K8: now also N?. (dpR), N?. (dpR), N?. (dpR), N?. (dpR), N?. (dpR), N?. (dpR), U?.1 (~{Q8}), U?.1 (~{Q8}), U?.1 (~{Q8}), U?.1 (~{Q8}), U?.1 (~{Q8})
- net K7: now reaches U?.10 (~{Q7})
- net K7: now also N?. (dpR), N?. (dpR), N?. (dpR), N?. (dpR), N?. (dpR), N?. (dpR), U?.10 (~{Q7}), U?.10 (~{Q7}), U?.10 (~{Q7}), U?.10 (~{Q7}), U?.10 (~{Q7})
- net K6: now reaches U?.11 (~{Q6})
- net K6: now also N?. (dpR), N?. (dpR), N?. (dpR), N?. (dpR), N?. (dpR), N?. (dpR), U?.11 (~{Q6}), U?.11 (~{Q6}), U?.11 (~{Q6}), U?.11 (~{Q6}), U?.11 (~{Q6})
- net K4: now reaches U?.13 (~{Q4})
- net K4: now also N?. (dpR), N?. (dpR), N?. (dpR), N?. (dpR), N?. (dpR), N?. (dpR), U?.13 (~{Q4}), U?.13 (~{Q4}), U?.13 (~{Q4}), U?.13 (~{Q4}), U?.13 (~{Q4})
- net K5: now reaches U?.14 (~{Q5})
- net K5: now also N?. (dpR), N?. (dpR), N?. (dpR), N?. (dpR), N?. (dpR), N?. (dpR), U?.14 (~{Q5}), U?.14 (~{Q5}), U?.14 (~{Q5}), U?.14 (~{Q5}), U?.14 (~{Q5})
- net K1: now reaches U?.15 (~{Q1})
- net K1: now also N?. (dpR), N?. (dpR), N?. (dpR), N?. (dpR), N?. (dpR), N?. (dpR), U?.15 (~{Q1}), U?.15 (~{Q1}), U?.15 (~{Q1}), U?.15 (~{Q1}), U?.15 (~{Q1})
- net K0: now reaches U?.16 (~{Q0})
- net K0: now also N?. (dpR), N?. (dpR), N?. (dpR), N?. (dpR), N?. (dpR), N?. (dpR), U?.16 (~{Q0}), U?.16 (~{Q0}), U?.16 (~{Q0}), U?.16 (~{Q0}), U?.16 (~{Q0})
- net K2: now reaches U?.8 (~{Q2})
- net K2: now also N?. (dpR), N?. (dpR), N?. (dpR), N?. (dpR), N?. (dpR), N?. (dpR), U?.8 (~{Q2}), U?.8 (~{Q2}), U?.8 (~{Q2}), U?.8 (~{Q2}), U?.8 (~{Q2})
- net K3: now reaches U?.9 (~{Q3})
- net K3: now also N?. (dpR), N?. (dpR), N?. (dpR), N?. (dpR), N?. (dpR), N?. (dpR), U?.9 (~{Q3}), U?.9 (~{Q3}), U?.9 (~{Q3}), U?.9 (~{Q3}), U?.9 (~{Q3})
- net Left_Btn: no longer names the net of U?.29 (PC7)
- net Left_Btn: now also SW?.1
- net Middle_Btn: no longer names the net of U?.28 (PC6)
- net Middle_Btn: now also SW?.1
- net Right_Btn: no longer names the net of U?.27 (PC5)
- net Right_Btn: now also SW?.1
- new net: N?. (dpR), R?.1 (x5)
- no-connect marks 13 -> 19
Other:
- moved on the sheet: C?, J?, N?, R?, U?

Commit message: Schematic update
Parts:
- removed U?: DS1307+, Package_DIP:DIP-8_W7.62mm, symbol Timer_RTC:DS1307+
- added D? (x2): 1N4148, Diode_THT:D_DO-35_SOD27_P7.62mm_Horizontal, symbol Diode:1N4148
- added U?: PCF8583, symbol PCF8583:PCF8583
- Y?: value 32768Hz -> 32.768KHz
Connections:
- net GND: now also U?.3 (ADDR), U?.4 (GND)
- net OE: now also U?.13 (~{OE}), U?.13 (~{OE}), U?.13 (~{OE}), U?.4 (PB3); no longer U?.17 (PD3)
- net RCLK: now also U?.12 (RCLK), U?.12 (RCLK), U?.12 (RCLK)
- net SCL: now also R?.1, U?.6 (SCL)
- net SDA: now also R?.1, U?.5 (SDA)
- net SRCLK: now also U?.11 (SRCLK), U?.11 (SRCLK), U?.11 (SRCLK)
- net SRCLR: now also U?.10 (~{SRCLR}), U?.10 (~{SRCLR}), U?.10 (~{SRCLR})
- net VCC: now also U?.16 (VCC), D?.2 (A)
- net at Y?.1: now also U?.2 (X2)
- net at Y?.2: now also U?.1 (X1)
- net at Li-Po.1 (+): now also D?.2 (A)
- net Data renamed DATA
- new net: D?.1 (K), D?.1 (K), U?.8 (VCC)
- no-connect marks 19 -> 20
Other:
- moved on the sheet: Li-Po, R?, Y?

Commit message: Schematic update
Parts:
- added J?: AVR-ISP-10, symbol Connector:AVR-ISP-10
Connections:
- net GND: now also J?.10 (GND), J?.4 (GND), J?.6 (GND), J?.8 (GND)
- net MOSI: now reaches U?.6 (PB5)
- net MOSI: now also J?.1 (MOSI)
- net MISO: now reaches U?.7 (PB6)
- net MISO: now also J?.9 (MISO)
- net SCK: now reaches U?.8 (PB7)
- net SCK: now also J?.7 (SCK)
- net RST: now reaches R?.2, U?.9 (~{RESET})
- net RST: now also J?.5 (~{RST})
- no-connect marks 20 -> 21
Changed lines of the file:
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@@
   (junction (at 72.39 171.45) (diameter 0) (color 0 0 0 0)
   )
+  (junction (at 34.29 34.29) (diameter 0) (color 0 0 0 0)
+  )
   (junction (at 92.71 87.63) (diameter 0) (color 0 0 0 0)
   )
@@
   (no_connect (at 259.08 81.28))
   (no_connect (at 184.15 88.9))
+  (no_connect (at 153.67 158.75))
   (no_connect (at 184.15 121.92))
   (no_connect (at 184.15 40.64))
@@
     (stroke (width 0) (type default) (color 0 0 0 0))
   )
+  (wire (pts (xy 34.29 27.94) (xy 34.29 34.29))
+    (stroke (width 0) (type default) (color 0 0 0 0))
+  )
   (wire (pts (xy 276.86 76.2) (xy 279.4 76.2))
     (stroke (width 0) (type default) (color 0 0 0 0))
@@
     (stroke (width 0) (type default) (color 0 0 0 0))
   )
+  (wire (pts (xy 153.67 181.61) (xy 153.67 182.88))
+    (stroke (width 0) (type default) (color 0 0 0 0))
+  )
   (wire (pts (xy 172.72 114.3) (xy 176.53 114.3))
     (stroke (width 0) (type default) (color 0 0 0 0))
@@
     (stroke (width 0) (type default) (color 0 0 0 0))
   )
+  (wire (pts (xy 64.77 74.93) (xy 66.04 74.93))
+    (stroke (width 0) (type default) (color 0 0 0 0))
+  )
   (bus (pts (xy 210.82 34.29) (xy 210.82 38.1))
     (stroke (width 0) (type default) (color 0 0 0 0))
@@
     (stroke (width 0) (type default) (color 0 0 0 0))
   )
+  (wire (pts (xy 64.77 72.39) (xy 66.04 72.39))
+    (stroke (width 0) (type default) (color 0 0 0 0))
+  )
   (wire (pts (xy 247.65 71.12) (xy 251.46 71.12))
     (stroke (width 0) (type default) (color 0 0 0 0))
@@
     (stroke (width 0) (type default) (color 0 0 0 0))
   )
+  (wire (pts (xy 64.77 69.85) (xy 66.04 69.85))
+    (stroke (width 0) (type default) (color 0 0 0 0))
+  )
   (wire (pts (xy 127 162.56) (xy 132.08 162.56))
     (stroke (width 0) (type default) (color 0 0 0 0))
@@
     )
   )
+  (global_label "MISO" (shape input) (at 66.04 72.39 0) (fields_autoplaced)
+    (effects (font (size 1.27 1.27)) (justify left))
+    (property "Intersheet References" "${INTERSHEET_REFS}" (id 0) (at 73.0493 72.3106 0)
+      (effects (font (size 1.27 1.27)) (justify left) hide)
+    )
+  )
   (global_label "SRCLR" (shape input) (at 106.68 71.12 180) (fields_autoplaced)
     (effects (font (size 1.27 1.27)) (justify right))
@@
     )
   )
+  (global_label "SCK" (shape input) (at 166.37 171.45 0) (fields_autoplaced)
+    (effects (font (size 1.27 1.27)) (justify left))
+    (property "Intersheet References" "${INTERSHEET_REFS}" (id 0) (at 172.5326 171.3706 0)
+      (effects (font (size 1.27 1.27)) (justify left) hide)
+    )
+  )
   (global_label "DATA" (shape input) (at 106.68 63.5 180) (fields_autoplaced)
     (effects (font (size 1.27 1.27)) (justify right))
@@
     )
   )
+  (global_label "RST" (shape input) (at 34.29 27.94 90) (fields_autoplaced)
+    (effects (font (size 1.27 1.27)) (justify left))
+    (property "Intersheet References" "${INTERSHEET_REFS}" (id 0) (at 34.2106 22.0798 90)
+      (effects (font (size 1.27 1.27)) (justify left) hide)
+    )
+  )
   (global_label "SRCLR" (shape input) (at 106.68 114.3 180) (fields_autoplaced)
     (effects (font (size 1.27 1.27)) (justify right))
@@
     )
   )
+  (global_label "MOSI" (shape input) (at 66.04 69.85 0) (fields_autoplaced)
+    (effects (font (size 1.27 1.27)) (justify left))
+    (property "Intersheet References" "${INTERSHEET_REFS}" (id 0) (at 73.0493 69.7706 0)
+      (effects (font (size 1.27 1.27)) (justify left) hide)
+    )
+  )
+  (global_label "MOSI" (shape input) (at 166.37 168.91 0) (fields_autoplaced)
+    (effects (font (size 1.27 1.27)) (justify left))
+    (property "Intersheet References" "${INTERSHEET_REFS}" (id 0) (at 173.3793 168.8306 0)
+      (effects (font (size 1.27 1.27)) (justify left) hide)
+    )
+  )
   (global_label "HV" (shape input) (at 261.62 25.4 0) (fields_autoplaced)
     (effects (font (size 1.27 1.27)) (justify left))
@@
     )
   )
+  (global_label "SCK" (shape input) (at 66.04 74.93 0) (fields_autoplaced)
+    (effects (font (size 1.27 1.27)) (justify left))
+    (property "Intersheet References" "${INTERSHEET_REFS}" (id 0) (at 72.2026 74.8506 0)
+      (effects (font (size 1.27 1.27)) (justify left) hide)
+    )
+  )
   (global_label "HV" (shape input) (at 186.69 25.4 0) (fields_autoplaced)
     (effects (font (size 1.27 1.27)) (justify left))
@@
     )
   )
+  (global_label "MISO" (shape input) (at 166.37 166.37 0) (fields_autoplaced)
+    (effects (font (size 1.27 1.27)) (justify left))
+    (property "Intersheet References" "${INTERSHEET_REFS}" (id 0) (at 173.3793 166.2906 0)
+      (effects (font (size 1.27 1.27)) (justify left) hide)
+    )
+  )
   (global_label "SRCLK" (shape input) (at 106.68 111.76 180) (fields_autoplaced)
     (effects (font (size 1.27 1.27)) (justify right))
@@
     )
   )
+  (global_label "RST" (shape input) (at 166.37 173.99 0) (fields_autoplaced)
+    (effects (font (size 1.27 1.27)) (justify left))
+    (property "Intersheet References" "${INTERSHEET_REFS}" (id 0) (at 172.2302 173.9106 0)
+      (effects (font (size 1.27 1.27)) (justify left) hide)
+    )
+  )
   (global_label "SCL" (shape input) (at 76.2 36.83 180) (fields_autoplaced)
     (effects (font (size 1.27 1.27)) (justify right))
@@
     (pin "1")
   )
+  (symbol (lib_id "power:GND") (at 153.67 182.88 0) (unit 1)
+    (in_bom yes) (on_board yes)
+    (property "Reference" "#PWR?" (id 0) (at 153.67 189.23 0)
+      (effects (font (size 1.27 1.27)) hide)
+    )
+    (property "Value" "GND" (id 1) (at 154.94 186.69 0))
+    (property "Footprint" "" (id 2) (at 153.67 182.88 0)
+      (effects (font (size 1.27 1.27)) hide)
+    )
+    (property "Datasheet" "" (id 3) (at 153.67 182.88 0)
+      (effects (font (size 1.27 1.27)) hide)
+    )
+    (pin "1")
+  )
   (symbol (lib_id "ITT5870S:ITT5870S") (at 267.97 69.85 0) (unit 1)
     (in_bom yes) (on_board yes)
@@
     (pin "1")
   )
+  (symbol (lib_id "Connector:AVR-ISP-10") (at 156.21 171.45 0) (unit 1)
+    (in_bom yes) (on_board yes)
+    (property "Reference" "J?" (id 0) (at 166.37 179.07 0)
+      (effects (font (size 1.27 1.27)) (justify right))
+    )
+    (property "Value" "AVR-ISP-10" (id 1) (at 166.37 181.61 0)
+      (effects (font (size 1.27 1.27)) (justify right))
+    )
+    (property "Footprint" "" (id 2) (at 149.86 170.18 90)
+      (effects (font (size 1.27 1.27)) hide)
+    )
+    (property "Datasheet" " ~" (id 3) (at 123.825 185.42 0)
+      (effects (font (size 1.27 1.27)) hide)
+    )
+    (pin "1")
+    (pin "10")
+    (pin "2")
+    (pin "3")
+    (pin "4")
+    (pin "5")
+    (pin "6")
+    (pin "7")
+    (pin "8")
+    (pin "9")
+  )
   (symbol (lib_id "Device:R_Small") (at 29.21 34.29 90) (unit 1)
     (in_bom yes) (on_board yes)
@@
       (reference "#PWR?") (unit 1) (value "GND") (footprint "")
     )
+    (path "/710e33b0-8ab7-4d57-b20d-41aa95d940fd"
+      (reference "#PWR?") (unit 1) (value "GND") (footprint "")
+    )
     (path "/7f35a441-260b-499c-9ce6-6ec1bc2b6cdc"
       (reference "#PWR?") (unit 1) (value "VCC") (footprint "")
@@
       (reference "J?") (unit 1) (value "Jack-DC") (footprint "")
     )
+    (path "/e70f1643-9a68-4811-928a-039a5b29791e"
+      (reference "J?") (unit 1) (value "AVR-ISP-10") (footprint "")
+    )
     (path "/51b5addd-22e0-4282-a9f3-004c98e0d2f0"
